File: SPI Bus Buffer/eagle/SPI Bus Buffer/SPI Bus Buffer.sch (EAGLE design)
At the start: 33 parts, among them IC1 74LS541N

Commit message: Update: Eagel files of the SPI Bus Buffer
Parts:
- added JP6: OUT3, pinhead:PINHD-1X8
- added JP7: OUT4, pinhead:PINHD-1X8
- added JP8: OUT5, pinhead:PINHD-1X8
- added JP9: IN2, pinhead:PINHD-1X8
- added R16: 33, rcl:R-EU_0207/7
- added TP2: TPPAD1-13, testpad:TPPAD1-13
- JP1: value IN -> IN1; device pinhead:PINHD-1X7 -> pinhead:PINHD-1X8
- JP2: value OUT -> OUT1; device pinhead:PINHD-1X7 -> pinhead:PINHD-1X8
- JP4: device pinhead:PINHD-1X7 -> pinhead:PINHD-1X8
- R15: value 1k -> 470
Connections:
- removed net O_LDAC_DCA: JP2.5, JP4.5, R4.2
- new net N$16: IC1A.Y4, R16.1
- new net N$17: JP5.9, LED1.C, LED2.C, LED3.C, LED4.C, LED5.C, LED6.C, LED7.C, LED8.C
- new net O_LDCA_DCA: JP2.7, JP4.7, JP6.7, JP7.7, JP8.7, R5.2
- new net O_RESET: JP2.8, JP4.8, JP6.8, JP7.8, JP8.8, R6.2
- new net RESET: IC1A.A7, JP1.8, JP9.8
- net CS_DCA: now also IC1A.A5, JP1.6, JP9.6; no longer IC1A.A1, JP1.1
- net CS_DCF: now also IC1A.A4, JP1.5, JP9.5; no longer IC1A.A7, JP1.7
- net CS_DCO: now also IC1A.A3, JP1.4, JP9.4; no longer IC1A.A6, JP1.6
- net GND: now also JP1.1, JP2.1, JP4.1, JP6.1, JP7.1, JP8.1, JP9.1, TP2.TP; no longer IC1A.A4, JP1.4, JP2.4, JP4.4, JP5.9, LED1.C, LED2.C, LED3.C, LED4.C, LED5.C, LED6.C, LED7.C, LED8.C
- net LDAC_DCA: now also IC1A.A6, JP1.7, JP9.7; no longer IC1A.A5, JP1.5
- net MOSI: now also IC1A.A2, JP9.3; no longer IC1A.A3
- net O_CS_DCA: now also JP2.6, JP4.6, JP6.6, JP7.6, JP8.6, R4.2; no longer JP2.1, JP4.1, R1.2
- net O_CS_DCF: now also JP2.5, JP4.5, JP6.5, JP7.5, JP8.5, R16.2; no longer JP2.7, JP4.7, R6.2
- net O_CS_DCO: now also JP2.4, JP4.4, JP6.4, JP7.4, JP8.4, R3.2; no longer JP2.6, JP4.6, R5.2
- net O_MOSI: now also JP6.3, JP7.3, JP8.3, R2.2; no longer R3.2
- net O_SCK: now also JP6.2, JP7.2, JP8.2, R1.2; no longer R2.2
- net SCK: now also IC1A.A1, JP9.2; no longer IC1A.A2
Other:
- moved on the sheet: TP1
