File: 5V_3.3V_+-2.5V_PowerSupply/eagle/+5V_3.3V_+-2.5V_PowerSupply.sch (EAGLE design)
At the start: 55 parts, among them IC1 7805TV, IC2 LM4558N, IC3 TA48033S, SW1 PUSH_SW_ALT

Commit message: Update: 5V_3V3_2V5_PowerSupply Eagle Files
Parts:
- removed SL1: PWRIN+, con-amp-quick:M02
- removed SL2: PWRIN-, con-amp-quick:M02
- removed U$1, U$2: POLYSWITCH, mylib2:POLYSWITCH
- added JP21: TP_GND, pinhead:PINHD-1X2
- added PS1, PS2: POLYSWITCH-5,0, mylib2:POLYSWITCH-5,0
- added X1: PWR-, con-wago-500:W237-102
- added X2: PWR+, con-wago-500:W237-102
- C1, C11, C2: device rcl:C-EU050-025X075 -> rcl:C-EU025-024X044
- C10, C9: device rcl:CPOL-EUE2.5-6 -> rcl:CPOL-EUE2.5-7
- C5: device rcl:C-EU050-024X044 -> rcl:C-EU025-024X044
- IC2: value LM4558N -> LM4556
- JP15, JP17, JP18, JP3, JP4: value +3.3V -> +2.5V
- LED1, LED4, LED5: value (none) -> GREEN
- LED2: value (none) -> RED
- LED3: value (none) -> BLUE
Connections:
- new net V+: C1.2, C2.1, C4.-, C6.+, IC2A.-IN, IC2A.OUT, JP15.1, JP17.1, JP18.1, JP3.1, JP4.1, LED5.A
- net +3V3: no longer C1.2, C2.1, C4.-, C6.+, IC2A.-IN, IC2A.OUT, JP15.1, JP17.1, JP18.1, JP3.1, JP4.1, LED5.A
- net +9V: now also JP19.1, JP20.1, R2.1; no longer LED2.A
- net -9V: now also JP19.3, JP20.3
- net GND: now also JP19.2, JP20.2, JP21.1, JP21.2, LED2.C, X1-1.KL, X2-2.KL; no longer R2.2, SL1.1, SL2.2
- net N$1: now also PS2.2, X2-1.KL; no longer SL2.1, U$2.2
- net N$10: now also PS1.2, X1-2.KL; no longer SL1.2, U$1.2
- net N$11: now also PS2.1, SW1.P; no longer SW1.P1, U$2.1
- net N$2: now also PS1.1, SW1.P1; no longer SW1.P, U$1.1
- net N$4: now also LED2.A, R2.2; no longer LED2.C, R2.1
Other:
- moved on the sheet: JP10, JP11, JP12, JP13, JP14, JP15, JP17, JP18, JP3, JP4, JP5, JP6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

Commit message: Update: Eagle files
Parts:
- removed JP16, JP19, JP20: +-9V, pinhead:PINHD-1X3
- removed JP17, JP18: +2.5V, pinhead:PINHD-1X2
- JP10, JP9: value +3.3V -> +5V_2V5; device pinhead:PINHD-1X2 -> pinhead:PINHD-1X3
- JP13: value +5V -> +3.3V
- JP15: value +2.5V -> +3.3V
- JP3, JP4: value +2.5V -> +-9V; device pinhead:PINHD-1X2 -> pinhead:PINHD-1X3
- JP5: value +5V -> +-9V; device pinhead:PINHD-1X2 -> pinhead:PINHD-1X3
- JP6, JP7, JP8: value +5V -> +5V_2V5; device pinhead:PINHD-1X2 -> pinhead:PINHD-1X3
Connections:
- net +3V3: now also JP13.1, JP15.1; no longer JP10.1, JP9.1
- net +5V: now also JP10.1, JP9.1; no longer JP13.1, JP5.1
- net +9V: now also JP3.1, JP4.1, JP5.1; no longer JP16.1, JP19.1, JP20.1
- net -9V: now also JP3.3, JP4.3, JP5.3; no longer JP16.3, JP19.3, JP20.3
- net GND: now also JP10.3, JP6.3, JP7.3, JP8.3, JP9.3; no longer JP10.2, JP16.2, JP17.2, JP18.2, JP19.2, JP20.2, JP6.2, JP7.2, JP8.2, JP9.2
- net V+: now also JP10.2, JP6.2, JP7.2, JP8.2, JP9.2; no longer JP15.1, JP17.1, JP18.1, JP3.1, JP4.1
Other:
- moved on the sheet: JP11, JP12, JP13, JP14, JP15, JP21
