File: BaseMachine Exio Board/eagle/BaseMachine_Exio_Board/BaseMachine_Exio_Board.brd (EAGLE design)
At the start: 73.3 x 48.2 mm, 15 parts, among them IC1 MCP23S17SP, IC2 AT24CP

Commit message: Update: BaseMachine Exio Board
Parts:
- added R4: 1k, rcl:0207/7
Connections:
- net GND: now also R4.1
- net MISO: now also R4.2
Routing:
- net GND: track 175.3 -> 177.8 mm
Other:
- board text added: "Do not connect"
Changed lines of the file:
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@@
 <layer number="97" name="Info" color="7" fill="1" visible="no" active="no"/>
 <layer number="98" name="Guide" color="6" fill="1" visible="no" active="no"/>
-<layer number="100" name="Grid" color="11" fill="1" visible="yes" active="yes"/>
-<layer number="101" name="PWR_LINE" color="7" fill="1" visible="yes" active="yes"/>
+<layer number="100" name="Grid" color="11" fill="1" visible="no" active="yes"/>
+<layer number="101" name="PWR_LINE" color="7" fill="1" visible="no" active="yes"/>
 <layer number="200" name="200bmp" color="1" fill="10" visible="no" active="no"/>
 <layer number="201" name="tNamesOnPCB" color="5" fill="1" visible="yes" active="yes"/>
@@
 <hole x="69.85" y="44.45" drill="3.2"/>
 <hole x="69.85" y="3.81" drill="3.2"/>
+<text x="33.02" y="43.18" size="1.778" layer="48">Do not connect</text>
+<wire x1="30.48" y1="29.21" x2="40.64" y2="43.18" width="0" layer="48"/>
+<wire x1="40.64" y1="43.18" x2="48.26" y2="43.18" width="0" layer="48"/>
 </plain>
 <attributes>
@@
 <element name="JP5" library="pinhead" package="1X09/90" value="LOAD_SAVE" x="20.32" y="34.29"/>
 <element name="JP6" library="pinhead" package="1X02" value="TP_GND" x="5.08" y="24.13" rot="R90"/>
+<element name="R4" library="rcl" package="0207/7" value="1k" x="60.96" y="19.05" rot="R270"/>
 </elements>
 <signals>
@@
 <wire x1="5.08" y1="25.4" x2="7.62" y2="25.4" width="1.016" layer="16"/>
 <wire x1="5.08" y1="22.86" x2="7.62" y2="22.86" width="1.016" layer="16"/>
+<contactref element="R4" pad="1"/>
+<wire x1="60.96" y1="22.86" x2="58.42" y2="22.86" width="1.016" layer="16"/>
 </signal>
 <signal name="+3V3">
@@
 <contactref element="IC1" pad="14"/>
 <contactref element="JP2" pad="4"/>
-<wire x1="68.58" y1="15.24" x2="43.18" y2="15.24" width="0.4064" layer="16"/>
 <wire x1="43.18" y1="20.32" x2="43.18" y2="15.24" width="0.4064" layer="16"/>
+<contactref element="R4" pad="2"/>
+<wire x1="43.18" y1="15.24" x2="60.96" y2="15.24" width="0.4064" layer="16"/>
+<wire x1="60.96" y1="15.24" x2="68.58" y2="15.24" width="0.4064" layer="16"/>
 </signal>
 <signal name="MOSI">
