File: BaseMachine Exio Board/eagle/BaseMachine_Exio_Board/BaseMachine_Exio_Board.sch (EAGLE design)
At the start: 15 parts, among them IC1 MCP23S17SP, IC2 AT24CP

Commit message: Update: BaseMachine Exio Board
Parts:
- added R4: 1k, rcl:R-EU_0207/7
Connections:
- net GND: now also R4.1
- net MISO: now also R4.2
Other:
- moved on the sheet: IC1, JP1, JP5
