File: BaseMachine Exio Board/eagle/BaseMachine_Exio_Board/BaseMachine_Exio_Load_Save.brd (EAGLE design)
At the start: 70.8 x 45.7 mm, 8 parts, among them SW1 AK_TCTSW, SW2 AK_TCTSW, SW3 AK_TCTSW, SW4 AK_TCTSW, SW5 AK_TCTSW, SW6 AK_TCTSW

Commit message: Update: BaseMachine Exio Board
Connections:
- removed net N$9: SW5.4
- net GND: now also SW5.4
Routing:
- net GND: track 159.6 -> 179.9 mm
Changed lines of the file:
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@@
 <wire x1="66.04" y1="33.02" x2="66.04" y2="7.62" width="1.016" layer="16"/>
 <wire x1="66.04" y1="7.62" x2="63.5" y2="5.08" width="1.016" layer="16"/>
-<wire x1="38.1" y1="30.48" x2="38.1" y2="33.02" width="1.016" layer="16"/>
+<wire x1="35.56" y1="33.02" x2="38.1" y2="33.02" width="1.016" layer="16"/>
 <wire x1="38.1" y1="33.02" x2="50.8" y2="33.02" width="1.016" layer="16"/>
 <wire x1="50.8" y1="33.02" x2="63.5" y2="33.02" width="1.016" layer="16"/>
@@
 <wire x1="50.8" y1="30.48" x2="50.8" y2="33.02" width="1.016" layer="16"/>
 <wire x1="63.5" y1="30.48" x2="63.5" y2="33.02" width="1.016" layer="16"/>
-</signal>
-<signal name="N$9">
 <contactref element="SW5" pad="4"/>
+<wire x1="35.56" y1="33.02" x2="35.56" y2="17.78" width="1.016" layer="16"/>
+<wire x1="35.56" y1="17.78" x2="38.1" y2="17.78" width="1.016" layer="16"/>
+<wire x1="38.1" y1="30.48" x2="38.1" y2="33.02" width="1.016" layer="16"/>
 </signal>
 </signals>
