File: BaseMachine Exio Board/eagle/BaseMachine_Exio_Board/BaseMachine_Exio_Load_Save.sch (EAGLE design)
At the start: 8 parts, among them SW1 AK_TCTSW, SW2 AK_TCTSW, SW3 AK_TCTSW, SW4 AK_TCTSW, SW5 AK_TCTSW, SW6 AK_TCTSW

Commit message: Update: BaseMachine Exio Board
Connections:
- removed net N$9: SW5.S@1
- net GND: now also SW5.S@1
Changed lines of the file:
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@@
 <pinref part="JP1" gate="A" pin="9"/>
 <label x="78.74" y="83.82" size="1.778" layer="95"/>
-</segment>
-</net>
-<net name="N$9" class="0">
-<segment>
 <pinref part="SW5" gate="G$1" pin="S@1"/>
 <wire x1="170.18" y1="104.14" x2="172.72" y2="104.14" width="0.1524" layer="91"/>
